Commit message: refined muscle display with partially correct muscle xml

File: examples/08-skeleton/human.urdf (robot description, URDF)
Before this commit: robot humanoid_clean, 40 links, 39 joints
Links:
- added link base, mass 1.0
- added link chest, mass 0.1
Joints:
- added joint pelvis_base_fixed: type fixed, parent pelvis, child base, origin xyz=0 0 0 rpy=0 0 0
- added joint torso_chest_fixed: type fixed, parent torso, child chest, origin xyz=0 0 0 rpy=0 0 0
